File: PCB/tivaAdapterPcb.brd (EAGLE design)
At the start: 134.6 x 32.7 mm, 4 parts

Commit message: route
Parts:
- moved TIVA2 76.1 mm to (30.6, 59.0), flipped to the bottom
- moved ARRAY_SENSOR 60.2 mm to (99.4, 43.4), flipped to the bottom
- moved LCD 54.7 mm to (43.1, 43.8)
- moved TIVA1 46.0 mm to (91.7, 58.9), flipped to the bottom
Connections:
- new net 3V3_1: TIVA1.2
- new net 5V_1: TIVA1.1
- net 3V3: no longer TIVA1.2
- net 5V: no longer TIVA1.1
Routing:
- net PF2: track 0.00 -> 76.7 mm, vias 0 -> 1
- net PF3: track 0.00 -> 75.6 mm, vias 0 -> 1
- net PF1: track 0.00 -> 75.5 mm, vias 0 -> 1
- net PF0: track 0.00 -> 74.1 mm
- net PM4: track 0.00 -> 60.3 mm
- net PM5: track 0.00 -> 54.8 mm
- net PN3: track 0.00 -> 50.1 mm
- net PL3: track 0.00 -> 49.3 mm
- net PM6: track 0.00 -> 48.9 mm
- net PM3: track 0.00 -> 46.4 mm
- net PN2: track 0.00 -> 44.9 mm
- net PM7: track 0.00 -> 44.2 mm
- net PM2: track 0.00 -> 40.8 mm
- net PN0: track 0.00 -> 37.7 mm, vias 0 -> 1
- net PM1: track 0.00 -> 35.3 mm
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- added copper zone on layer 16, net GND
Other:
- board text added: "3V3"
- board text added: "5V"
- board text added: "BachelorProjekt-Ole-Hung"
- board text added: "CS"
- board text added: "DB0"
- board text added: "DB1"
- board text added: "DB10"
- board text added: "DB11"
- board text added: "DB12"
- board text added: "DB13"
- board text added: "DB15"
- board text added: "DB2"
- board text added: "DB3"
- board text added: "DB4"
- board text added: "DB5"
- board text added: "DB6"
- board text added: "DB7"
- board text added: "DB8"
- board text added: "DB9"
- board text added: "F_CS"
- board text added: "GND"
- board text added: "LED_A"
- board text added: "NC"
- board text added: "PD0"
- board text added: "PD1"
- board text added: "PD2"
- board text added: "PD3"
- board text added: "PD4"
- board text added: "PD5"
- board text added: "PD6"
- board text added: "PD7"
- board text added: "PE2"
- board text added: "PE3"
- board text added: "PE4"
- board text added: "PE5"
- board text added: "PF0"
- board text added: "PF1"
- board text added: "PF2"
- board text added: "PF3"
- board text added: "PK0"
- board text added: "PK1"
- board text added: "PK2"
- board text added: "PK3"
- board text added: "RD"
- board text added: "RESET"
- board text added: "RS"
- board text added: "SD_CLK"
- board text added: "SD_CS"
- board text added: "SD_D0"
- board text added: "SD_DIN"
- board text added: "T_CLK"
- board text added: "T_CS"
- board text added: "T_D0"
- board text added: "T_DIN"
- board text added: "T_IQR"
- board text added: "VREF"
- board text added: "WR"
