File: PCB/tivaAdapterPcb.sch (EAGLE design)
At the start: 4 parts

Commit message: route
Connections:
- new net 3V3_1: TIVA1.2
- new net 5V_1: TIVA1.1
- net 3V3: no longer TIVA1.2
- net 5V: no longer TIVA1.1
Other:
- moved on the sheet: ARRAY_SENSOR
